File: PCB/geigercCounter_pcb.kicad_pcb (KiCad board)
At the start: 2 copper layers, 150 x 98.2 mm, 96 parts, among them J1 Molex Micro Fit, J2 Debugpins, J3 USB-TYPE-C-018, J4 Femal Connector for LCD I2C b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, Q1 IRLML6402TRPBF, Q2 BCW68, Q3 PBHV8560Z, Q4 MMBT3904, Q5 MMBT3904, SW1 GPIO4, SW2 GPIO5, SW3 Reset, SW4 Boot, SW5 SW_SPDT, U1 TPS631000DRLR, U2 MCP73871-2AA, U3 ESP32-S3-WROOM-1_multi_unit, U4 ICM7555IBAZ

Commit message: 10.08.2025 Layout Version 0.2
Parts:
- removed the D8 at (126.5, 58.8)
- removed the R19 at (144.2, 124.9)
- removed the R21 at (125.5, 112.2)
- added ?: , clipboard:ea0946bf-12c1-49c3-a260-f9acbf49f04f, F.Cu at (143.1, 69.3)
- added D13: D_Small, Diode_SMD:D_SOD-323_HandSoldering, F.Cu at (207.1, 78.7)
- added R15: 10k, Resistor_SMD:R_0805_2012Metric_Pad1.20x1.40mm_HandSolder, F.Cu at (177.7, 77.5)
- added R20: 560k, Resistor_SMD:R_0805_2012Metric_Pad1.20x1.40mm_HandSolder, F.Cu at (161.8, 65.2)
- added R22: 10k, Resistor_SMD:R_0805_2012Metric_Pad1.20x1.40mm_HandSolder, F.Cu at (148.5, 59.5)
- added REF**: MountingHole_3.5mm_Pad_Via, MountingHole:MountingHole_3.5mm_Pad_Via, F.Cu at (147.2, 70.0)
- added REF**: MountingHole_3.5mm_Pad_Via, MountingHole:MountingHole_3.5mm_Pad_Via, F.Cu at (126.5, 56.8)
- D9: value 3,3V Good -> PWR
- moved BZ1 174.7 mm to (225.7, 51.2), turned to 180 degrees
- moved R29 157.9 mm to (221.8, 53.2), turned to 90 degrees
- moved D1 152.1 mm to (218.8, 57.5), turned to -90 degrees
- moved D2 146.6 mm to (218.8, 60.5), turned to -90 degrees
- moved Q4 141.8 mm to (218.8, 53.0), turned to 90 degrees
- moved C16 132.3 mm to (100.7, 48.1)
- moved R28 128.3 mm to (96.8, 41.2)
- moved R30 127.2 mm to (96.8, 43.2), turned to 0 degrees
- moved R26 127.2 mm to (207.8, 56.8), turned to 180 degrees
- moved R23 126.7 mm to (196.6, 46.9), turned to 180 degrees
- moved R27 124.7 mm to (104.5, 42.8)
- moved Q5 120.2 mm to (100.6, 43.9), turned to -90 degrees
- moved R21 119.3 mm to (192.8, 46.9), turned to 180 degrees
- moved C14 119.1 mm to (195.8, 50.5), turned to 90 degrees
- moved D19 117.1 mm to (187.9, 42.2), turned to 180 degrees
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- renumbered D13 to D14, D14 to D15, D15 to D16, D16 to D17, D17 to D18, D18 to D19, R15 to R16, R16 to R17, R17 to R18, R18 to R19, R20 to R21, R22 to R23, R23 to R24, R24 to R25, R25 to R26, R26 to R27, R27 to R28, R28 to R29, R29 to R30, R30 to R31, R31 to R32, R32 to R33, R33 to R34
Connections:
- net Net-(D10-K) renamed GPIO3
- J2 pad 5: GPIO8 -> I_L_HV
- J2 pad 6: Vhigh/100 -> Trig_HV
- J2 pad 7: Trig_HV -> Vhigh/100
- J2 pad 8: I_L_HV -> GPIO1
- R10 pad 1: Net-(U3A-GPIO10) -> Net-(U3A-GPIO9)
- R11 pad 1: Net-(U3A-GPIO11) -> Net-(U3A-GPIO10)
- R26 pad 2: GPIO12 -> GPIO11
- SW1 pad 1: Net-(U3A-GPIO10) -> Net-(U3A-GPIO9)
- SW1 pad 3: Net-(U3A-GPIO10) -> Net-(U3A-GPIO9)
- SW2 pad 1: Net-(U3A-GPIO11) -> Net-(U3A-GPIO10)
- SW2 pad 3: Net-(U3A-GPIO11) -> Net-(U3A-GPIO10)
- U3 pad 15: Vhigh/100 -> Net-(D13-A)
- U3 pad 17: GPIO9 -> Net-(U3A-GPIO9)
- U3 pad 19: Net-(U3A-GPIO11) -> GPIO11
- U3 pad 38: unconnected-(U3B-GPIO2-Pad38) -> Vhigh/100
- U4 pad 4: GPIO9 -> GPIO12
Routing:
- net UART0_TX: track 4.34 -> 154.9 mm, vias 0 -> 3
- net (no net): track 121.4 -> 0.00 mm, vias 4 -> 0
- net Net-(D13-A): track 0.00 -> 118.6 mm
- net GPIO11: track 0.00 -> 117.0 mm
- net UART0_RX: track 37.8 -> 151.7 mm, vias 1 -> 3
- net Net-(U3A-GPIO9): track 0.00 -> 109.9 mm, vias 0 -> 2
- net GPIO1: track 60.4 -> 165.9 mm, vias 2 -> 3
- net Net-(U3A-GPIO10): track 26.7 -> 116.3 mm, vias 1 -> 0
- net Vbat_USB: track 177.8 -> 100.7 mm, vias 7 -> 4
- net D-: track 239.1 -> 170.5 mm, vias 5 -> 3
- net GPIO16/U0CTS: track 64.7 -> 133.2 mm, vias 2 -> 3
- net D+: track 232.2 -> 167.8 mm, vias 3 -> 1
- net GPIO15/U0RTS: track 72.5 -> 135.8 mm, vias 2 -> 3
- net GPIO12: track 12.9 -> 66.3 mm
- net Net-(U3A-EN): track 79.0 -> 25.7 mm, vias 2 -> 0
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- added copper zone on F.Cu, net +3.3V
- added copper zone on B.Cu, net GND
- added copper zone on F.Cu, net GND
- added copper zone on F.Cu, net Vbat_USB
- removed copper zone on F.Cu, net VBUS
Other:
- board size 150 x 98.2 mm -> 150 x 43 mm
- board text added: "Geiger-Müller-Zählrohr"
- board text added: "High Voltage Do Not Touch!"
- board text added: "Jonas Stelzeneder"

Commit message: Bestellversion
Parts:
- removed the Q3 at (178.0, 50.5)
- removed the R21 at (192.8, 46.9)
- removed the R31 at (186.8, 51.2)
- removed the R32 at (186.8, 55.0)
- added C18: 10nF 200V, Capacitor_SMD:C_0805_2012Metric_Pad1.18x1.45mm_HandSolder, F.Cu at (189.2, 58.2)
- added C19: 10nF 200V, Capacitor_SMD:C_0805_2012Metric_Pad1.18x1.45mm_HandSolder, F.Cu at (189.2, 54.5)
- added C20: 10nF 200V, Capacitor_SMD:C_0805_2012Metric_Pad1.18x1.45mm_HandSolder, F.Cu at (180.5, 49.0)
- added C22: 10nF 200V, Capacitor_SMD:C_0805_2012Metric_Pad1.18x1.45mm_HandSolder, F.Cu at (189.5, 50.2)
- added D20: PNE20010, Diode_SMD:Nexperia_CFP3_SOD-123W, F.Cu at (185.9, 53.9)
- added D21: PNE20010, Diode_SMD:Nexperia_CFP3_SOD-123W, F.Cu at (183.7, 50.9)
- added D22: PNE20010, Diode_SMD:Nexperia_CFP3_SOD-123W, F.Cu at (184.9, 47.4)
- added D23: PNE20010, Diode_SMD:Nexperia_CFP3_SOD-123W, F.Cu at (189.5, 47.4)
- added JP3: SolderJumper_2_Open, Jumper:SolderJumper-2_P1.3mm_Open_RoundedPad1.0x1.5mm, F.Cu at (150.6, 44.0)
- added Q1: IRLML6344, Package_TO_SOT_SMD:SOT-23-3, F.Cu at (110.4, 49.5)
- added Q4: PBHV8560Z, Package_TO_SOT_SMD:SOT-223-3_TabPin2, F.Cu at (173.0, 53.5)
- added R17: 100R, Resistor_SMD:R_0805_2012Metric_Pad1.20x1.40mm_HandSolder, B.Cu at (223.6, 79.1)
- added R24: 1M, Resistor_SMD:R_0805_2012Metric_Pad1.20x1.40mm_HandSolder, F.Cu at (193.6, 47.3)
- added R34: 1M, Resistor_SMD:R_0805_2012Metric_Pad1.20x1.40mm_HandSolder, F.Cu at (158.0, 43.0)
- added R35: 1M, Resistor_SMD:R_0805_2012Metric_Pad1.20x1.40mm_HandSolder, F.Cu at (154.2, 44.0)
- added R6: 100R, Resistor_SMD:R_0805_2012Metric_Pad1.20x1.40mm_HandSolder, F.Cu at (114.8, 50.4)
- C17: value 10nF 1kV -> 10nF 200V; footprint Capacitor_SMD:C_1206_3216Metric_Pad1.33x1.80mm_HandSolder -> Capacitor_SMD:C_0805_2012Metric_Pad1.18x1.45mm_HandSolder
- D13: value D_Small -> 1N4148WS
- D18: value RS1M -> PNE20010; footprint Diode_SMD:D_SMA -> Diode_SMD:Nexperia_CFP3_SOD-123W
- D9: value PWR -> 3V3 PWR
- L2: footprint CustomLib:Inductor_wuerth_74404086103 -> CustomLib:Inductor_wuerth_7447709222; moved to B.Cu
- SW1: value GPIO4 -> GPIO9
- SW2: value GPIO5 -> GPIO10
- moved L2 49.8 mm to (219.4, 46.8), turned to 180 degrees
- moved R33 26.1 mm to (162.0, 41.8)
- moved ? 20.0 mm to (123.2, 71.0)
- moved R36 16.1 mm to (145.7, 45.0)
- moved C21 14.8 mm to (147.8, 45.0)
- moved C17 11.5 mm to (180.5, 53.0), turned to 90 degrees
- moved D18 11.0 mm to (185.9, 58.5), turned to -90 degrees
- moved D14 7.42 mm to (167.0, 48.5), turned to -90 degrees
- moved D15 2.26 mm to (167.0, 44.5), turned to -90 degrees
- moved D16 1.68 mm to (170.0, 43.0)
- moved D17 1.68 mm to (177.0, 43.0)
- moved D19 1.63 mm to (186.5, 43.0)
- moved Q2 1.40 mm to (214.4, 71.8), turned to 90 degrees
- moved JP1 1.25 mm to (209.2, 73.1)
- moved R10 1.25 mm to (211.5, 72.8)
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- renumbered C15 to C14, C14 to C15, C18 to C21, Q1 to Q2, Q2 to Q3, Q4 to Q5, Q5 to Q6, R9 to R10, R10 to R11, R11 to R12, R12 to R13, R13 to R14, R14 to R15, R15 to R16, R16 to R18, R17 to R19, R18 to R20, R19 to R21, R20 to R22, R22 to R23, R23 to R25, R24 to R26, R25 to R27, R26 to R28, R27 to R29, R28 to R30, R29 to R31, R30 to R32, R34 to R36, R6 to R7, R7 to R8, R8 to R9
Connections:
- C17 pad 1: Vhigh -> Net-(D18-A)
- C17 pad 2: GND -> Net-(D20-K)
- C8 pad 1: Net-(Q1-S) -> Net-(Q2-S)
- D18 pad 1: Vhigh -> Net-(D18-K)
- J4 pad 1: GND -> Net-(J4-Pin_1)
- Q2 pad 1: Vbat_USB -> Net-(Q2-G)
- Q2 pad 2: Net-(Q1-G) -> Net-(Q2-S)
- Q2 pad 3: Net-(Q1-S) -> Vbat_USB
- R15 pad 1: Net-(Q1-S) -> Net-(Q2-S)
- R15 pad 2: Net-(Q1-G) -> Net-(Q2-G)
- R33 pad 1: Net-(R32-Pad2) -> Vhigh
- R33 pad 2: Vhigh/100 -> Net-(R33-Pad2)
- SW5 pad 2: Net-(Q1-G) -> Net-(SW5-B)
- U2 pad 1: Net-(Q1-S) -> Net-(Q2-S)
- U2 pad 20: Net-(Q1-S) -> Net-(Q2-S)
- U3 pad 23: unconnected-(U3B-GPIO21-Pad23) -> GPIO21
Routing:
- net I_L_HV: track 54.2 -> 112.4 mm, vias 2 -> 4
- net Vhigh/100: track 113.2 -> 73.9 mm, vias 3 -> 1
- net Net-(D18-A): track 21.6 -> 57.1 mm, vias 0 -> 1
- net Vhigh: track 14.5 -> 38.2 mm
- net Net-(Q1-G): track 25.1 -> 1.78 mm, vias 1 -> 0
- net Net-(Q2-G): track 0.00 -> 20.9 mm, vias 0 -> 1
- net GPIO21: track 0.00 -> 18.6 mm
- net Net-(Q2-S): track 0.00 -> 14.6 mm
- net +3.3V: track 187.8 -> 199.4 mm
- net Net-(D21-K): track 0.00 -> 10.8 mm
- net Net-(D22-K): track 0.00 -> 10.8 mm
- net Net-(D18-K): track 0.00 -> 9.91 mm
- net Net-(Q1-S): track 9.71 -> 0.00 mm
- net Net-(Q4-B): track 18.7 -> 27.4 mm
- net GND: track 216.9 -> 225.0 mm, vias 58 -> 50
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- removed copper zone on F.Cu, net GND
Other:
- outline, holes or cut-outs redrawn
- board text added: "Geiger-Müller-Zählrohr V1.0"
- board text removed: "Geiger-Müller-Zählrohr"
