File: PCB/geigercCounter_pcb.kicad_sch (KiCad schematic)
At the start: 95 parts, among them J1 Molex Micro Fit, J2 Debugpins, J3 USB-TYPE-C-018, J4 Femal Connector for LCD I2C b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, Q1 IRLML6402TRPBF, Q2 BCW68, Q3 PBHV8560Z, Q4 MMBT3904, Q5 MMBT3904, SW1 GPIO4, SW2 GPIO5, SW3 Reset, SW4 Boot, SW5 SW_SPDT, U1 TPS631000DRLR, U2 MCP73871-2AA, U3 ESP32-S3-WROOM-1_multi_unit, U4 ICM7555IBAZ

Commit message: 10.08.2025 Layout Version 0.2
Parts:
- added D13: D_Small, Diode_SMD:D_SOD-323_HandSoldering, symbol Device:D_Small
- added R15: 10k, Resistor_SMD:R_0805_2012Metric_Pad1.20x1.40mm_HandSolder, symbol Device:R_Small
- R22: renamed from R21; value 100k -> 10k
- renumbered D13 to D14, D14 to D15, D15 to D16, D16 to D17, D17 to D18, D18 to D19, R15 to R16, R16 to R17, R17 to R18, R18 to R19, R19 to R20, R20 to R21, R22 to R23, R23 to R24, R24 to R25, R25 to R26, R26 to R27, R27 to R28, R28 to R29, R29 to R30, R30 to R31, R31 to R32, R32 to R33, R33 to R34
Connections:
- net GPIO8 is gone; now on net I_L_HV: J2.5 (Pin_5)
- net +3.3V: now also R15.1
- net GPIO1: now also J2.8 (Pin_8)
- net GPIO12: now also R22.1, U4.4 (~{R}); no longer R26.2
- net I_L_HV: no longer J2.8 (Pin_8)
- net Trig_HV: now also J2.6 (Pin_6); no longer J2.7 (Pin_7)
- net Vhigh/100: now also J2.7 (Pin_7), U3.38 (GPIO2/ADC1_CH1); no longer J2.6 (Pin_6), U3.15 (GPIO3/ADC1_CH2)
- net at R10.1, SW1.1, SW1.3 (1): now also U3.17 (GPIO9); no longer U3.18 (GPIO10)
- net at R11.1, SW2.1, SW2.3 (1): now also U3.18 (GPIO10); no longer U3.19 (GPIO11)
- net GPIO3: now reaches D10.1 (K), U2.6 (~{PG})
- net GPIO3: now also D13.1 (K)
- removed net GPIO9: R22.1, U3.17 (GPIO9), U4.4 (~{R})
- new net: D13.2 (A), R15.2, U3.15 (GPIO3)
- new net GPIO11: R26.2, U3.19 (GPIO11)
- no-connect marks 25 -> 23

Commit message: Bestellversion
Parts:
- removed D18: RS1M, Diode_SMD:D_SMA, symbol Device:D
- added C17, C19, C20, C22: 10nF 200V, Capacitor_SMD:C_0805_2012Metric_Pad1.18x1.45mm_HandSolder, symbol Device:C_Small
- added D18, D20, D21, D22, D23: PNE20010, Diode_SMD:Nexperia_CFP3_SOD-123W, symbol Device:D_Small
- added JP3: SolderJumper_2_Open, Jumper:SolderJumper-2_P1.3mm_Open_RoundedPad1.0x1.5mm, symbol Jumper:SolderJumper_2_Open
- added Q1: IRLML6344, Package_TO_SOT_SMD:SOT-23-3, symbol Simulation_SPICE:NMOS
- added R17, R6: 100R, Resistor_SMD:R_0805_2012Metric_Pad1.20x1.40mm_HandSolder, symbol Device:R_Small
- C18: renamed from C17; value 10nF 1kV -> 10nF 200V; footprint Capacitor_SMD:C_1206_3216Metric_Pad1.33x1.80mm_HandSolder -> Capacitor_SMD:C_0805_2012Metric_Pad1.18x1.45mm_HandSolder
- D13: value D_Small -> 1N4148WS
- D9: value 3,3V Good -> 3V3 PWR
- L2: footprint CustomLib:Inductor_wuerth_74404086103 -> CustomLib:Inductor_wuerth_7447709222
- SW1: value GPIO4 -> GPIO9
- SW2: value GPIO5 -> GPIO10
- renumbered C15 to C14, C14 to C15, C18 to C21, Q1 to Q2, Q2 to Q3, Q3 to Q4, Q4 to Q5, Q5 to Q6, R9 to R10, R10 to R11, R11 to R12, R12 to R13, R13 to R14, R14 to R15, R15 to R16, R16 to R18, R17 to R19, R18 to R20, R19 to R21, R20 to R22, R22 to R23, R21 to R24, R23 to R25, R24 to R26, R25 to R27, R26 to R28, R27 to R29, R28 to R30, R29 to R31, R30 to R32, R31 to R33, R32 to R34, R33 to R35, R34 to R36, R6 to R7, R7 to R8, R8 to R9
Connections:
- net GND: now also Q1.2 (S); no longer J4.1 (Pin_1)
- net Vbat_USB: now also Q2.3 (D); no longer Q2.1 (D)
- net Vhigh: now also C22.2, D23.1 (K); no longer C18.1
- net Vhigh/100: now also JP3.1 (A); no longer R35.2
- net at L2.2, Q4.2 (C): now also C17.1, D18.2 (A)
- net at C8.1, R15.1, U2.1 (OUT)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: now also Q2.2 (S); no longer Q2.3 (S)
- new net: Q1.1 (G), R6.2
- new net: J4.1 (Pin_1), Q1.3 (D)
- new net: JP3.2 (B), R35.2
- new net: C19.2, C22.1, D21.1 (K), D22.2 (A)
- new net: C18.1, C19.1, D18.1 (K), D20.2 (A)
- new net: Q2.1 (G), R15.2, R17.2
- new net: C17.2, C20.1, D20.1 (K), D21.2 (A)
- new net: C20.2, D22.1 (K), D23.2 (A)
- new net: R17.1, SW5.2 (B)
- new net GPIO21: R6.1, U3.23 (GPIO21)
- no-connect marks 23 -> 22
Other:
- moved on the sheet: BZ1, C12, C13, C14, C15, C16, C18, C21, D14, D15, D16, D17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
